File: DemoBoard/DemoBoard.kicad_pcb (KiCad board)
At the start: 2 copper layers, 45 x 45 mm, 58 parts, among them J1 USB4110GFA, J2 Conn_01x10_Pin, J3 Conn_01x10_Pin, J4 Conn_01x10_Pin, J5 Conn_01x10_Pin, SW1 SW_Push, SW2 SW_Push, U1 RP2040, U2 W25Q128JVSIM, U3 MCP2518FDT-E_QBB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

Commit message: Merging v0.1 to main (#1)
Parts:
- removed J2, J3, J4, J5: Conn_01x10_Pin, Connector_PinSocket_2.54mm:PinSocket_1x10_P2.54mm_Vertical
- removed JP1: 3, Jumper:SolderJumper-2_P1.3mm_Open_RoundedPad1.0x1.5mm
- removed JP2: 2, Jumper:SolderJumper-2_P1.3mm_Open_RoundedPad1.0x1.5mm
- removed JP3: 1, Jumper:SolderJumper-2_P1.3mm_Open_RoundedPad1.0x1.5mm
- removed JP4: 0, Jumper:SolderJumper-2_P1.3mm_Open_RoundedPad1.0x1.5mm
- added C24: 100nF, Capacitor_SMD:C_0402_1005Metric_Pad0.74x0.62mm_HandSolder, F.Cu at (143.6, 64.2)
- added C25: 47uF, Capacitor_SMD:C_1206_3216Metric_Pad1.33x1.80mm_HandSolder, F.Cu at (144.6, 45.6)
- added G***: LOGO, inspireFly:longInspireFly_12mmX4mm, F.Cu at (123.7, 67.1)
- added J6: M55-7101242R, inspireFly:HARWIN_M55-7101242R, F.Cu at (139.3, 39.8)
- added J7: MSD-1-A, inspireFly:CUI_MSD-1-A, F.Cu at (154.3, 63.2)
- added J8: Conn_01x17_Pin, Connector_PinSocket_2.54mm:PinSocket_1x17_P2.54mm_Vertical, F.Cu at (119.1, 75.9)
- added R11: 10k, Resistor_SMD:R_0402_1005Metric_Pad0.72x0.64mm_HandSolder, F.Cu at (143.6, 62.9)
- C22: footprint Capacitor_SMD:C_0402_1005Metric -> Capacitor_SMD:C_0402_1005Metric_Pad0.74x0.62mm_HandSolder
- C23: value 10uF -> 47uF; footprint Capacitor_SMD:C_0402_1005Metric -> Capacitor_SMD:C_1206_3216Metric_Pad1.33x1.80mm_HandSolder
- D1, D2, R8, R9: moved to B.Cu
- JP5: value SolderJumper_2_Open -> 3.3V EN; footprint Jumper:SolderJumper-2_P1.3mm_Open_RoundedPad1.0x1.5mm -> inspireFly:SmallJumper
- moved Y2 45.3 mm to (121.0, 43.6), turned to 180 degrees
- moved U4 42.0 mm to (127.2, 36.1)
- moved D2 40.7 mm to (123.2, 71.6)
- moved D1 40.3 mm to (123.3, 68.4)
- moved TP3 38.0 mm to (151.3, 37.1)
- moved TP2 36.8 mm to (154.4, 37.1)
- moved SW2 36.3 mm to (119.6, 52.3), turned to 90 degrees
- moved J1 34.7 mm to (155.2, 47.1), turned to 90 degrees
- moved R10 34.5 mm to (130.9, 36.4), turned to -90 degrees
- moved SW1 33.6 mm to (119.6, 59.4), turned to 90 degrees
- moved C22 33.1 mm to (148.9, 37.3), turned to 90 degrees
- moved R6 33.0 mm to (156.2, 39.9), turned to 180 degrees
- moved R7 29.9 mm to (120.2, 48.4), turned to 180 degrees
- moved U2 27.8 mm to (128.4, 51.2), turned to 45 degrees
- moved C2 27.0 mm to (136.1, 66.2)
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Connections:
- net SPI0_CS renamed SPI0_CS_CAN
- R8 pad 1: GPIO_5_DEBUGLED -> GPIO_6
- U1 pad 7: GPIO_5_DEBUGLED -> SPI0_CS_SDCARD
Routing:
- net CAN_HIGH: track 0.00 -> 61.4 mm, vias 0 -> 1
- net CAN_LOW: track 0.00 -> 59.8 mm, vias 0 -> 3
- net USB_VOLTAGE: track 0.00 -> 53.2 mm, vias 0 -> 1
- net +3.3V: track 0.00 -> 49.6 mm, vias 0 -> 20
- net GPIO_15: track 0.00 -> 42.9 mm, vias 0 -> 2
- net GPIO_14: track 0.00 -> 41.9 mm, vias 0 -> 2
- net SPI0_MOSI: track 0.00 -> 38.6 mm, vias 0 -> 4
- net SPI0_MISO: track 0.00 -> 38.2 mm, vias 0 -> 3
- net GPIO_9: track 0.00 -> 35.6 mm
- net ADC_3: track 0.00 -> 35.5 mm, vias 0 -> 1
- net SPI0_CLK: track 0.00 -> 34.7 mm, vias 0 -> 4
- net ADC_2: track 0.00 -> 34.0 mm, vias 0 -> 1
- net ADC_0: track 0.00 -> 33.8 mm, vias 0 -> 1
- net ADC_1: track 0.00 -> 33.5 mm, vias 0 -> 1
- net GPIO_17: track 0.00 -> 26.8 mm, vias 0 -> 2
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- added copper zone on F.Cu, net +3.3V
- added copper zone on In2.Cu, net +3.3V
- added copper zone on F.Cu, net BATTERY_VOLTAGE
- added copper zone on B.Cu, net GND
- added copper zone on F.Cu, net GND
- added copper zone on In1.Cu, net GND
- added copper zone on F.Cu, net USB_VOLTAGE
Other:
- copper layers 2 -> 4
- board text added: "BOOT0"
- board text added: "CAN L CAN H +3.3V SWCLK GND SWD USB_V A0 A1 A2 A3 9 14 15 16 17 GND"
- board text added: "Payload Demo Board"
- board text added: "RST"
