File: DemoBoard/DemoBoard.kicad_pcb (KiCad board)
At the start: 4 copper layers, 45 x 45 mm, 57 parts, among them J1 USB4110GFA, J6 M55-7101242R, J7 MSD-1-A, J8 Conn_01x17_Pin, SW1 SW_Push, SW2 SW_Push, U1 RP2040, U2 W25Q128JVSIM, U3 MCP2518FDT-E_QBB, U4 TCAN332DCNR, U5 TLV75533PDBVR, Y1 ABM8-272-T3, Y2 ABM8-20.000MHZ-10-B1U-T

Commit message: To be reviewed v0.2 to main (#4)
* Added R&D folders

* Add files via upload

* Delete Byte the Sky/Byte_The_Sky_smallBoard directory

* Add files via upload

* Add files via upload

* Add files via upload

* Add files via upload

* Add files via upload

* Add files via upload

* Add files via upload

* Add files via upload

* Add files via upload

* Add files via upload

* Add files via upload

* Add files via upload

* Delete Byte the Sky/inspireflybytetheskysmallboard/smallboard.kicad_sch

* Delete Byte the Sky/inspireflybytetheskysmallboard/smallboard.kicad_pro

* Delete Byte the Sky/inspireflybytetheskysmallboard/smallboard.kicad_pcb

* Add files via upload

* Add files via upload

* Add files via upload

* Add files via upload

* Add files via upload

* Add files via upload

* Updated BOM

* Add files via upload

* Add files via upload

* Add files via upload

* Add files via upload

* code

* Delete Flux and Radiation Tracker/inspireFly_F.A.R.T_BOM.xlsx

Replacing with updated BOM

* Updated BOM

* Add files via upload

Temperature sensor

* Add files via upload

* Add files via upload

* Updated DemoBoard to V0.2

* Fix silkscreen on Demoboard

* Update BOM for Demoboard

* Add files via upload

* Add files via upload

* Implement STM schematic

* Fix cap values for clock

* Fix cap values for clock

* added flash

* Routed capacitors

* schematic_added_flash

* Routing + schematic updates for STM

* Finalize STM payload + BOM

---------

Co-authored-by: Hsc2077 <146699419+Hsc2077@users.noreply.github.com>
Co-authored-by: Floating-Necc <meaneek.mandal@gmail.com>
Co-authored-by: byron11235813 <bmillet06@vt.edu>
Co-authored-by: JDRobertsNathan <jdroberts@vt.edu>
Co-authored-by: Christian G <tianvez273@gmail.com>
Co-authored-by: Matt-Scala <matthewscala3820@gmail.com>
Co-authored-by: Michael Karam <michaelkaram233@gmail.com>
Parts:
- removed U3: MCP2518FDT-E_QBB, inspireFly:SON65P450X300X90-15N
- added R12: 10k, Resistor_SMD:R_0402_1005Metric_Pad0.72x0.64mm_HandSolder, F.Cu at (130.5, 43.6)
- added U6: MCP2515T-I/ML, inspireFly:QFN20_4x4MC_MCH, F.Cu at (126.2, 42.5)
- C14, C15: value 18pF -> 15pF
- moved C17 1.37 mm to (130.5, 41.4)
- moved C15 0.22 mm to (119.5, 40.7)
- moved Y2 0.09 mm to (121.0, 43.7)
Connections:
- U1 pad 13: GPIO_10 -> SPI1_CLK
- U1 pad 14: GPIO_11 -> SPI1_MOSI
- U1 pad 15: GPIO_12 -> SPI1-MISO
- U1 pad 16: GPIO_13 -> SPI1_CS_CAN
- U1 pad 3: SPI0_CS_CAN -> GPIO_1
Routing:
- net SPI1_CS_CAN: track 0.00 -> 27.2 mm, vias 0 -> 2
- net SPI1-MISO: track 0.00 -> 24.0 mm, vias 0 -> 2
- net SPI0_CS_CAN: track 19.9 -> 0.00 mm, vias 2 -> 0
- net SPI1_MOSI: track 0.00 -> 19.8 mm, vias 0 -> 2
- net SPI1_CLK: track 0.00 -> 19.5 mm, vias 0 -> 2
- net SPI0_MOSI: track 38.6 -> 20.2 mm, vias 4 -> 2
- net SPI0_MISO: track 38.2 -> 21.0 mm, vias 3 -> 2
- net SPI0_CLK: track 34.7 -> 17.6 mm, vias 4 -> 2
- net GPIO_15: track 42.9 -> 34.9 mm
- net INT_CAN_CONTROLLER: track 20.6 -> 16.5 mm
- net Net-(U6-*RESET): track 0.00 -> 4.05 mm
- net +3.3V: track 49.6 -> 52.1 mm
- net Net-(U6-OSC1): track 8.86 -> 6.63 mm
- net Net-(U6-OSC2): track 8.87 -> 6.66 mm
- net GPIO_6: track 17.8 -> 19.9 mm
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Other:
- board text added: "Payload Demo Board V0.2"
- board text removed: "Payload Demo Board"
