File: Flux and Radiation Tracker/Flux_And_Radiation_Tracker_smallBoard/Flux_And_Radiation_Tracker_smallBoard.kicad_sch (KiCad schematic)
At the start: 14 parts, among them J1 Conn_01x07, U1 LTR-390UV-01, U2 MMC5983MA

Commit message: Add files via upload
Parts:
- U2: footprint MMC5983MA:MMC5983MA_MEM -> MMC5982MA:MMC5983MA_MEM
Changed lines of the file:
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@@
 			)
 		)
-		(property "Footprint" "MMC5983MA:MMC5983MA_MEM"
+		(property "Footprint" "MMC5982MA:MMC5983MA_MEM"
 			(at 167.64 49.53 0)
 			(effects
