File: Flux and Radiation Tracker/Flux_And_Radiation_Tracker_smallBoard/Flux_And_Radiation_Tracker_smallBoard.kicad_sch (KiCad schematic)
At the start: 14 parts, among them J1 Conn_01x07, U1 LTR-390UV-01, U2 MMC5983MA

Commit message: Add files via upload
Parts:
- removed 2.7k1: R, Resistor_SMD:R_0603_1608Metric, symbol Device:R
- removed C1: 4.7u, Capacitor_SMD:C_0603_1608Metric, symbol Device:C
- removed C2: 0.1u, Capacitor_SMD:C_0603_1608Metric, symbol Device:C
- removed R1, R3: 2.7k, Resistor_SMD:R_0603_1608Metric, symbol Device:R
- removed U1: LTR-390UV-01, LTR-390UV:SMD6_LTR-390UV-01_LTO, symbol LTR-390UV:LTR-390UV-01
- C3, C5, C6, C7: footprint Capacitor_SMD:C_0603_1608Metric -> Capacitor_SMD:C_0402_1005Metric
- C4: footprint Capacitor_SMD:C_0805_2012Metric -> Capacitor_SMD:C_0402_1005Metric
Connections:
- net 3V3 is gone; now on net +3.3V: J1.1 (Pin_1)
- net ICM_INT1: no longer names the net of MT1.4 (INT1/INT)
- net ICM_INT2: no longer names the net of MT1.9 (INT2)
- net LTR_INT: no longer names the net of J1.5 (Pin_5)
- net LTR_INT: no longer J1.7 (Pin_7)
- net MAG_INT: no longer names the net of J1.6 (Pin_6)
- net MAG_SDO: no longer names the net of U2.5 (SPI_SDO)
- net MMC_INT: no longer names the net of U2.15 (INT)
- no-connect marks 1 -> 8
Other:
- note removed: "I2C Address: 0x53"
- note removed: "UV/Light Sensor Module"
- moved on the sheet: C3, C4, C5, C6, C7, J1, MT1, U2

Commit message: Add files via upload
Parts:
- added R1, R2: 2.7k, Resistor_SMD:R_0402_1005Metric_Pad0.72x0.64mm_HandSolder, symbol Device:R
- added R3, R4: 10k, Resistor_SMD:R_0402_1005Metric_Pad0.72x0.64mm_HandSolder, symbol Device:R
- C3, C4, C5, C6, C7: footprint Capacitor_SMD:C_0402_1005Metric -> Capacitor_SMD:C_0402_1005Metric_Pad0.74x0.62mm_HandSolder
Connections:
- net +3.3V: now also R1.1, R2.1, R3.1, R4.1
- net I2C_SCL: now also R1.2, R4.2
- net I2C_SDA: now also R2.2, R3.2
Other:
- moved on the sheet: C3, C4, C5, C6, C7, MT1
