File: Flux and Radiation Tracker/Flux_And_Radiation_Tracker_smallBoard/Flux_And_Radiation_Tracker_smallBoard.kicad_sch (KiCad schematic)
At the start: 12 parts, among them J1 Conn_01x07, U2 MMC5983MA

Commit message: Add files via upload
Parts:
- removed J1: Conn_01x07, Connector_PinHeader_2.54mm:PinHeader_1x07_P2.54mm_Vertical, symbol Connector_Generic:Conn_01x07
- removed R1, R2: 2.7k, Resistor_SMD:R_0402_1005Metric_Pad0.72x0.64mm_HandSolder, symbol Device:R
- added H1, H2, H3, H4: MountingHole, MountingHole:MountingHole_2.5mm, symbol Mechanical:MountingHole
- added J1: Conn_01x06_Pin, Connector_PinHeader_2.54mm:PinHeader_1x06_P2.54mm_Vertical, symbol Connector:Conn_01x06_Pin
- added J2: Conn_01x04_Pin, Connector_PinHeader_2.54mm:PinHeader_1x04_P2.54mm_Vertical, symbol Connector:Conn_01x04_Pin
Connections:
- net +3.3V: now also J1.2 (Pin_2), J2.4 (Pin_4)
- net GND: now also J1.3 (Pin_3), J2.3 (Pin_3)
- net I2C_SCL: now also J1.4 (Pin_4), J2.2 (Pin_2)
- net I2C_SDA: now also J1.5 (Pin_5), J2.1 (Pin_1)
- no-connect marks 8 -> 7
