File: Flux and Radiation Tracker/Flux_And_Radiation_Tracker_smallBoard/Flux_And_Radiation_Tracker_smallBoard.kicad_pcb (KiCad board)
At the start: 2 copper layers, 0 parts

Commit message: Add files via upload
Parts:
- added 2.7k1: R, Resistor_SMD:R_0603_1608Metric, F.Cu at (141.2, 83.9)
- added C1: 4.7u, Capacitor_SMD:C_0603_1608Metric, F.Cu at (141.2, 86.4)
- added C2: 0.1u, Capacitor_SMD:C_0603_1608Metric, F.Cu at (141.2, 88.9)
- added C3: 1u, Capacitor_SMD:C_0603_1608Metric, F.Cu at (141.2, 91.5)
- added C4: 10u, Capacitor_SMD:C_0805_2012Metric, F.Cu at (150.0, 96.8)
- added C5: 0.1u, Capacitor_SMD:C_0603_1608Metric, F.Cu at (141.2, 94.0)
- added C6: 2.2u, Capacitor_SMD:C_0603_1608Metric, F.Cu at (141.2, 96.5)
- added C7: 10n, Capacitor_SMD:C_0603_1608Metric, F.Cu at (141.2, 99.0)
- added J1: Conn_01x07, Connector_PinHeader_2.54mm:PinHeader_1x07_P2.54mm_Vertical, F.Cu at (145.5, 85.0)
- added MT1: ICM-42670-P, ICM-42670-P:XDCR_ICM-42670-P, F.Cu at (150.5, 84.7)
- added R1: 2.7k, Resistor_SMD:R_0603_1608Metric, F.Cu at (141.2, 101.5)
- added R3: 2.7k, Resistor_SMD:R_0603_1608Metric, F.Cu at (141.2, 104.0)
- added U1: LTR-390UV-01, LTR-390UV:SMD6_LTR-390UV-01_LTO, F.Cu at (150.5, 93.5)
- added U2: MMC5983MA, MMC5982MA:MMC5983MA_MEM, F.Cu at (150.2, 89.2)
