File: Byte the Sky/inspireflybytetheskysmallboard/smallboard/smallboard.kicad_pcb (KiCad board)
At the start: 2 copper layers, 23.3 x 21.5 mm, 15 parts, among them IC1 N34TS04MT3ETG, J1 Conn_01x07_Pin, U2 LSM6DSV, U4 LIS2MDLTR

Commit message: Add files via upload
Parts:
- added C6: C, Capacitor_SMD:C_0402_1005Metric, F.Cu at (102.3, 75.7)
- added C7: 100nF, Capacitor_SMD:C_0402_1005Metric, F.Cu at (102.9, 63.5)
- added R6: 10k, Resistor_SMD:R_0402_1005Metric, F.Cu at (99.3, 71.4)
- added R7: 10k, Resistor_SMD:R_0402_1005Metric, F.Cu at (99.1, 73.9)
- added U3: OPA381, OPA381:MSOP08, F.Cu at (111.1, 62.2)
- D2: footprint VEMD:VEMD8083 -> footprints:VEMD8083
- IC1: footprint N34:SON50P300X200X80-9N -> footprints:SON50P300X200X80-9N
- U4: footprint LIS2MDLTR:PQFN50P200X200X70-12N -> footprints:PQFN50P200X200X70-12N
- moved C1 17.7 mm to (112.5, 75.9), turned to 180 degrees
- moved C2 15.4 mm to (110.4, 77.4), turned to 90 degrees
- moved R4 13.7 mm to (111.0, 72.6), turned to -90 degrees
- moved U4 12.8 mm to (110.1, 75.2), turned to -90 degrees
- moved C5 8.69 mm to (108.0, 76.1), turned to 90 degrees
- moved R5 8.10 mm to (107.6, 74.4)
- moved R2 7.43 mm to (100.1, 66.7)
- moved R1 7.06 mm to (105.7, 63.5), turned to 90 degrees
- moved R3 3.78 mm to (102.4, 66.7)
- moved C4 3.66 mm to (108.2, 69.6), turned to 90 degrees
- moved IC1 3.26 mm to (102.3, 73.6), turned to 180 degrees
- moved J1 1.68 mm to (95.1, 60.5)
- moved C3 1.33 mm to (107.5, 65.5), turned to 0 degrees
- moved U2 1.08 mm to (106.2, 68.1), turned to 90 degrees
- moved D2 0.58 mm to (103.6, 59.7), turned to 0 degrees
Connections:
- C3 pad 2: Net-(U2-VDD) -> GND
- C4 pad 1: Net-(U2-VDD_IO) -> GND
- D2 pad 1: +3.3V -> Net-(D2-K)
- D2 pad 2: ADC_0 -> +3.3V
- IC1 pad 9: unconnected-(IC1-EP-Pad9) -> GND
- R1 pad 1: ADC_0 -> Net-(D2-K)
- R1 pad 2: GND -> ADC_0
- U2 pad 5: Net-(U2-VDD_IO) -> +3.3V
- U2 pad 8: Net-(U2-VDD) -> +3.3V
Routing:
- net GPIO_17: track 28.6 -> 5.85 mm, vias 1 -> 0
- net GPIO_16: track 22.0 -> 6.69 mm, vias 1 -> 0
- net Net-(U2-SCX): track 16.6 -> 9.12 mm, vias 4 -> 0
- net GND: track 17.5 -> 24.5 mm, vias 2 -> 7
- net Net-(D2-K): track 0.00 -> 6.05 mm, vias 0 -> 2
- net GPIO_15: track 16.1 -> 10.9 mm, vias 1 -> 2
- net +3.3V: track 81.5 -> 77.6 mm, vias 3 -> 5
- net Net-(U2-VDD): track 3.68 -> 0.00 mm
- net GPIO_14: track 13.8 -> 11.4 mm, vias 1 -> 0
- net ADC_0: track 12.8 -> 14.7 mm, vias 1 -> 0
- net Net-(U4-VDD): track 2.47 -> 0.73 mm
- net Net-(U2-VDD_IO): track 1.65 -> 0.00 mm
- net Net-(U2-SDX): track 9.06 -> 7.86 mm, vias 2 -> 0
- net Net-(U4-VDD_IO): track 2.03 -> 1.16 mm
- added copper zone on B.Cu, net GND
- removed copper zone on F.Cu, net GND
Other:
- board size 23.3 x 21.5 mm -> 23.3 x 21.4 mm

Commit message: Add files via upload
Parts:
- removed R4, R5: 10k, Resistor_SMD:R_0402_1005Metric
- removed U4: LIS2MDLTR, footprints:PQFN50P200X200X70-12N
- added IC2: IIS2MDCTR, LIBIIS2M:IIS2MDCTR, F.Cu at (111.6, 75.4)
- C1, C3, C4, C7: footprint Capacitor_SMD:C_0402_1005Metric -> Capacitor_SMD:C_0402_1005Metric_Pad0.74x0.62mm_HandSolder
- C2: value 100nF -> 220nF; footprint Capacitor_SMD:C_0402_1005Metric -> Capacitor_SMD:C_0402_1005Metric_Pad0.74x0.62mm_HandSolder
- C5: value 220nF -> 100nF; footprint Capacitor_SMD:C_0402_1005Metric -> Capacitor_SMD:C_0402_1005Metric_Pad0.74x0.62mm_HandSolder
- C6: value C -> 100nF; footprint Capacitor_SMD:C_0402_1005Metric -> Capacitor_SMD:C_0402_1005Metric_Pad0.74x0.62mm_HandSolder
- D2: footprint footprints:VEMD8083 -> LIB_VEMD8083:VEMD8083
- IC1: footprint footprints:SON50P300X200X80-9N -> LIB_N34TS04MT3ETG:SON50P300X200X80-9N
- R1, R2, R3, R6, R7: footprint Resistor_SMD:R_0402_1005Metric -> Resistor_SMD:R_0402_1005Metric_Pad0.72x0.64mm_HandSolder
- U2: footprint footprints:LGA14-L_2P59X3P1X0P5_STM -> ul_LSM6DSV:LGA14-L_2P59X3P1X0P5_STM
- U3: footprint OPA381:MSOP08 -> OPA381:OPA381 Amplifier
- moved C5 6.84 mm to (114.7, 74.9)
- moved C1 3.45 mm to (112.4, 72.5), turned to 90 degrees
- moved C2 2.51 mm to (107.9, 76.8), turned to 0 degrees
- moved U3 0.46 mm to (110.6, 62.2), turned to 0 degrees
Connections:
- C1 pad 1: +3.3V -> Net-(IC2-VDD_IO)
- C1 pad 2: Net-(U4-VDD_IO) -> +3.3V
- C2 pad 1: +3.3V -> GND
- C5 pad 1: GND -> Net-(IC2-VDD)
- C5 pad 2: Net-(U4-C1) -> +3.3V
Routing:
- net Net-(D2-K): track 6.05 -> 11.3 mm
- net +3.3V: track 77.6 -> 81.6 mm, vias 5 -> 6
- net Net-(IC2-C1): track 0.73 -> 4.15 mm
- net Net-(IC2-VDD): track 0.00 -> 2.51 mm
- net Net-(IC2-SDA/SDI/SDO): track 7.86 -> 9.74 mm
- net Net-(U4-C1): track 1.67 -> 0.00 mm
- net Net-(IC2-VDD_IO): track 0.00 -> 1.56 mm
- net Net-(IC2-SCL/SPC): track 9.12 -> 7.70 mm
- net Net-(U4-VDD_IO): track 1.16 -> 0.00 mm
- net GND: track 24.5 -> 25.3 mm, vias 7 -> 8

Commit message: Add files via upload
Parts:
- removed U3: OPA381, OPA381:OPA381 Amplifier
- added C8: 10uF, Capacitor_SMD:C_0402_1005Metric_Pad0.74x0.62mm_HandSolder, F.Cu at (114.0, 69.8)
- added U1: OPA381, OPA381AIDGKR:SOP65P490X110-8N, F.Cu at (112.3, 61.7)
- C7: value 100nF -> 10pF
- U2: value LSM6DSV -> LSM6
- moved C1 2.63 mm to (112.3, 69.9)
- moved C5 2.11 mm to (114.5, 72.8)
- moved C4 1.25 mm to (108.8, 70.6)
- moved C3 0.82 mm to (107.8, 64.8)
Connections:
- C1 pad 1: Net-(IC2-VDD_IO) -> +3.3V
- C1 pad 2: +3.3V -> GND
- C5 pad 1: Net-(IC2-VDD) -> +3.3V
- C5 pad 2: +3.3V -> GND
- IC2 pad 10: Net-(IC2-VDD_IO) -> +3.3V
- IC2 pad 9: Net-(IC2-VDD) -> +3.3V
Routing:
- net GND: track 25.3 -> 1.52 mm, vias 8 -> 5
- net +3.3V: track 81.6 -> 95.2 mm, vias 6 -> 8
- net Net-(D2-K): track 11.3 -> 19.0 mm
- net ADC_0: track 14.7 -> 19.5 mm
- net Net-(IC2-VDD): track 2.51 -> 0.00 mm
- net Net-(IC2-VDD_IO): track 1.56 -> 0.00 mm
- added copper zone on F.Cu, net GND
Other:
- board text added: "+"
- board text added: "-"

Commit message: Add files via upload
Parts:
- U1: value OPA381 -> OPA381AIDGKR
- U2: value LSM6 -> LSM6DSV
Routing:
- net +3.3V: track 95.2 -> 97.8 mm, vias 8 -> 9
Changed lines of the file:
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@@
 			)
 		)
-		(property "Value" "OPA381"
+		(property "Value" "OPA381AIDGKR"
 			(at -0.95 2.39 90)
 			(layer "F.Fab")
@@
 			)
 		)
-		(property "Value" "LSM6"
+		(property "Value" "LSM6DSV"
 			(at 0.8311 3.499999 90)
 			(unlocked yes)
@@
 	(footprint "Capacitor_SMD:C_0402_1005Metric_Pad0.74x0.62mm_HandSolder"
 		(layer "F.Cu")
-		(at 112.32 69.87 90)
+		(at 112.35 69.8875 90)
 		(descr "Capacitor SMD 0402 (1005 Metric), square (rectangular) end terminal, IPC-7351 nominal with elongated pad for handsoldering. (Body size source: IPC-SM-782 page 76, https://www.pcb-3d.com/wordpress/wp-content/uploads/ipc-sm-782a_amendment_1_and_2.pdf), generated with kicad-footprint-generator")
 		(tags "capacitor handsolder")
@@
 	(footprint "Capacitor_SMD:C_0402_1005Metric_Pad0.74x0.62mm_HandSolder"
 		(layer "F.Cu")
-		(at 113.96 69.8425 90)
+		(at 113.99 69.86 90)
 		(descr "Capacitor SMD 0402 (1005 Metric), square (rectangular) end terminal, IPC-7351 nominal with elongated pad for handsoldering. (Body size source: IPC-SM-782 page 76, https://www.pcb-3d.com/wordpress/wp-content/uploads/ipc-sm-782a_amendment_1_and_2.pdf), generated with kicad-footprint-generator")
 		(tags "capacitor handsolder")
@@
 	)
 	(segment
+		(start 112.32 72.76)
+		(end 112.32 70.485)
+		(width 0.4)
+		(layer "F.Cu")
+		(net 1)
+	)
+	(segment
 		(start 105.222901 67.581101)
 		(end 104.919101 67.581101)
@@
 	)
 	(segment
-		(start 113.8625 72.76)
-		(end 114.5 73.3975)
-		(width 0.4)
-		(layer "F.Cu")
-		(net 1)
-	)
-	(segment
 		(start 106.900002 66.387002)
 		(end 106.68 66.167)
@@
 	)
 	(segment
-		(start 110.65 70.28)
-		(end 112.1625 70.28)
+		(start 104.919101 67.581101)
+		(end 103.886 66.548)
 		(width 0.4)
 		(layer "F.Cu")
@@
 	)
 	(segment
-		(start 104.919101 67.581101)
-		(end 103.886 66.548)
+		(start 108.341099 68.581099)
+		(end 107.077101 68.581099)
 		(width 0.4)
 		(layer "F.Cu")
@@
 	)
 	(segment
-		(start 108.341099 68.581099)
-		(end 107.077101 68.581099)
+		(start 112.32 70.485)
+		(end 112.35 70.455)
 		(width 0.4)
 		(layer "F.Cu")
@@
 	)
 	(segment
-		(start 112.34 70.4575)
-		(end 112.32 70.4375)
+		(start 112.37 70.475)
+		(end 112.35 70.455)
 		(width 0.203)
 		(layer "F.Cu")
@@
 	)
 	(segment
-		(start 112.1625 70.28)
-		(end 112.32 70.4375)
+		(start 112.1925 70.2975)
+		(end 112.35 70.455)
 		(width 0.4)
 		(layer "F.Cu")
@@
 	)
 	(segment
-		(start 112.32 70.4375)
-		(end 113.9325 70.4375)
+		(start 112.35 70.455)
+		(end 113.9625 70.455)
 		(width 0.4)
 		(layer "F.Cu")
@@
 	)
 	(segment
-		(start 112.32 72.76)
-		(end 113.8625 72.76)
+		(start 98.298 66.167)
+		(end 100.076 66.167)
 		(width 0.4)
 		(layer "F.Cu")
@@
 	)
 	(segment
-		(start 98.298 66.167)
-		(end 100.076 66.167)
+		(start 108.85 69.09)
+		(end 108.341099 68.581099)
 		(width 0.4)
 		(layer "F.Cu")
@@
 	)
 	(segment
-		(start 108.85 69.09)
-		(end 108.341099 68.581099)
+		(start 113.96 75.11)
+		(end 112.7875 75.11)
+		(width 0.4)
+		(layer "F.Cu")
+		(net 1)
+	)
+	(segment
+		(start 113.98 75.13)
+		(end 113.96 75.11)
 		(width 0.4)
 		(layer "F.Cu")
@@
 	)
 	(segment
-		(start 113.9325 70.4375)
-		(end 113.96 70.41)
+		(start 113.9625 70.455)
+		(end 113.99 70.4275)
 		(width 0.4)
 		(layer "F.Cu")
@@
 	)
 	(segment
-		(start 112.28 70.4775)
-		(end 112.32 70.4375)
+		(start 112.31 70.495)
+		(end 112.35 70.455)
 		(width 0.203)
 		(layer "F.Cu")
@@
 	)
 	(via
+		(at 113.98 75.13)
+		(size 0.45)
+		(drill 0.3)
+		(layers "F.Cu" "B.Cu")
+		(net 1)
+	)
+	(via
 		(at 110.65 70.28)
 		(size 0.45)
@@
 	)
 	(segment
+		(start 112.32 72.76)
+		(end 113.98 74.42)
+		(width 0.4)
+		(layer "B.Cu")
+		(net 1)
+	)
+	(segment
 		(start 98.96 65.505)
 		(end 98.298 66.167)
@@
 		(width 0.4)
 		(layer "B.Cu")
+		(net 1)
+	)
+	(segment
+		(start 113.98 74.42)
+		(end 113.98 75.13)
+		(width 0.4)
+		(layer "B.Cu")

Commit message: Add files via upload
Parts:
- moved C8 1.46 mm to (114.8, 68.7)
Routing:
- net +3.3V: track 97.8 -> 101.7 mm
Changed lines of the file:
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@@
 	(footprint "Capacitor_SMD:C_0402_1005Metric_Pad0.74x0.62mm_HandSolder"
 		(layer "F.Cu")
-		(at 113.99 69.86 90)
+		(at 114.82 68.66 90)
 		(descr "Capacitor SMD 0402 (1005 Metric), square (rectangular) end terminal, IPC-7351 nominal with elongated pad for handsoldering. (Body size source: IPC-SM-782 page 76, https://www.pcb-3d.com/wordpress/wp-content/uploads/ipc-sm-782a_amendment_1_and_2.pdf), generated with kicad-footprint-generator")
 		(tags "capacitor handsolder")
@@
 	)
 	(segment
+		(start 113.49 69.94)
+		(end 114.2025 69.2275)
+		(width 0.4)
+		(layer "F.Cu")
+		(net 1)
+	)
+	(segment
 		(start 109.65 75.63)
 		(end 110.82 75.63)
@@
 		(start 103.886 66.548)
 		(end 103.886 66.167)
+		(width 0.4)
+		(layer "F.Cu")
+		(net 1)
+	)
+	(segment
+		(start 114.5 73.3975)
+		(end 113.47 72.3675)
 		(width 0.4)
 		(layer "F.Cu")
@@
 	)
 	(segment
-		(start 112.35 70.455)
-		(end 113.9625 70.455)
-		(width 0.4)
-		(layer "F.Cu")
-		(net 1)
-	)
-	(segment
 		(start 103.886 66.167)
 		(end 105.918 66.167)
@@
 	)
 	(segment
-		(start 113.9625 70.455)
-		(end 113.99 70.4275)
-		(width 0.4)
-		(layer "F.Cu")
-		(net 1)
-	)
-	(segment
 		(start 108.85 70.065)
 		(end 108.84 70.075)
@@
 	)
 	(segment
+		(start 113.47 72.3675)
+		(end 113.47 69.94)
+		(width 0.4)
+		(layer "F.Cu")
+		(net 1)
+	)
+	(segment
 		(start 105.918 66.167)
 		(end 105.918 66.1245)
@@
 		(start 100.838 75.692)
 		(end 100.838 74.398)
+		(width 0.4)
+		(layer "F.Cu")
+		(net 1)
+	)
+	(segment
+		(start 114.2025 69.2275)
+		(end 114.82 69.2275)
 		(width 0.4)
 		(layer "F.Cu")
@@
 		(layer "F.Cu")
 		(net 1)
+	)
+	(segment
+		(start 113.47 69.94)
+		(end 113.49 69.94)
+		(width 0.4)
+		(layer "F.Cu")
+		(net 1)
