File: Byte the Sky/inspireflybytetheskysmallboard/smallboard/smallboard.kicad_sch (KiCad schematic)
At the start: 15 parts, among them IC1 N34TS04MT3ETG, J1 Conn_01x07_Pin, U2 LSM6DSV, U4 LIS2MDLTR

Commit message: Add files via upload
Parts:
- removed C4: 100nF, Capacitor_SMD:C_0402_1005Metric, symbol Device:C_US
- added C4, C7: 100nF, Capacitor_SMD:C_0402_1005Metric, symbol Device:C
- added C6: 100 nF, Capacitor_SMD:C_0402_1005Metric, symbol Device:C
- added R6, R7: 10k, Resistor_SMD:R_0402_1005Metric, symbol Device:R
- added U3: OPA381, OPA381:MSOP08, symbol Device:Opamp_Dual
- C3: symbol Device:C_US -> Device:C
- D2: footprint VEMD:VEMD8083 -> footprints:VEMD8083
- IC1: footprint N34:SON50P300X200X80-9N -> footprints:SON50P300X200X80-9N
- U4: footprint LIS2MDLTR:PQFN50P200X200X70-12N -> footprints:PQFN50P200X200X70-12N
Connections:
- net +3.3V: now also D2.2 (A), U2.5 (VDD_IO), U2.8 (VDD), C4.2, C6.2, R6.1, R7.1; no longer D2.1 (K)
- net ADC_0: now also R1.2, C7.2, U3.1; no longer D2.2 (A), R1.1
- net GND: now also C3.2, IC1.9 (EP), C4.1, C6.1, U3.2 (-); no longer R1.2
- net GPIO_16: now also R6.2
- net GPIO_17: now also R7.2
- new net: C7.1, D2.1 (K), R1.1, U3.3 (+)
- no-connect marks 10 -> 9
Other:
- moved on the sheet: C1, C2, C3, C5, D2, IC1, R1, R2, R3

Commit message: Add files via upload
Parts:
- removed C1, C2: 100nF, Capacitor_SMD:C_0402_1005Metric, symbol Device:C_US
- removed C5: 220nF, Capacitor_SMD:C_0402_1005Metric, symbol Device:C_US
- removed R4, R5: 10k, Resistor_SMD:R_0402_1005Metric, symbol Device:R
- removed U4: LIS2MDLTR, footprints:PQFN50P200X200X70-12N, symbol LIS2MDLTR:LIS2MDLTR
- added C1, C5: 100nF, Capacitor_SMD:C_0402_1005Metric_Pad0.74x0.62mm_HandSolder, symbol Device:C
- added C2: 220nF, Capacitor_SMD:C_0402_1005Metric_Pad0.74x0.62mm_HandSolder, symbol Device:C
- added IC2: IIS2MDCTR, LIBIIS2M:IIS2MDCTR, symbol IIS2MDCTR:IIS2MDCTR
- C3, C4, C7: footprint Capacitor_SMD:C_0402_1005Metric -> Capacitor_SMD:C_0402_1005Metric_Pad0.74x0.62mm_HandSolder
- C6: value 100 nF -> 100nF; footprint Capacitor_SMD:C_0402_1005Metric -> Capacitor_SMD:C_0402_1005Metric_Pad0.74x0.62mm_HandSolder
- D2: footprint footprints:VEMD8083 -> LIB_VEMD8083:VEMD8083
- IC1: footprint footprints:SON50P300X200X80-9N -> LIB_N34TS04MT3ETG:SON50P300X200X80-9N
- R1, R2, R3, R6, R7: footprint Resistor_SMD:R_0402_1005Metric -> Resistor_SMD:R_0402_1005Metric_Pad0.72x0.64mm_HandSolder
- U2: footprint footprints:LGA14-L_2P59X3P1X0P5_STM -> ul_LSM6DSV:LGA14-L_2P59X3P1X0P5_STM
- U3: footprint OPA381:MSOP08 -> OPA381:OPA381 Amplifier
Connections:
- net +3.3V: now also C1.2, C5.2, IC2.3 (CS)
- net GND: now also C2.1, IC2.6 (GND_1), IC2.8 (GND_2)
- net at U2.2 (SDX): now also IC2.4 (SDA/SDI/SDO)
- net at U2.3 (SCX): now also IC2.1 (SCL/SPC)
- new net: C1.1, IC2.10 (VDD_IO)
- new net: C2.2, IC2.5 (C1)
- new net: C5.1, IC2.9 (VDD)

Commit message: Add files via upload
Parts:
- removed U3: OPA381, OPA381:OPA381 Amplifier, symbol Device:Opamp_Dual
- added C8: 10uF, Capacitor_SMD:C_0402_1005Metric_Pad0.74x0.62mm_HandSolder, symbol Device:C
- added U1: OPA381AIDGKR, OPA381AIDGKR:SOP65P490X110-8N, symbol OPA381AIDGKR:OPA381AIDGKR
Connections:
- net +3.3V: now also C1.1, C5.1, IC2.10 (VDD_IO), IC2.9 (VDD), C8.1, U1.7 (V+); no longer C1.2, C5.2
- net ADC_0: now also U1.6 (OUT)
- net GND: now also C1.2, C5.2, C8.2, U1.3 (+IN), U1.4 (V-)
- net at C7.1, D2.1 (K), R1.1: now also U1.2 (-IN)
Other:
- moved on the sheet: C1, C5, C7, D2, R1

Commit message: Add files via upload
Parts:
- C7: value 100nF -> 10pF
Changed lines of the file:
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@@
 			)
 		)
-		(property "Value" "100nF"
+		(property "Value" "10pF"
 			(at 222.25 107.95 90)
 			(effects

Commit message: Add files via upload
Other:
- moved on the sheet: C8
Changed lines of the file:
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@@
-	)
-	(junction
-		(at 130.81 99.06)
-		(diameter 0)
-		(color 0 0 0 0)
 	)
 	(junction
@@
 	)
 	(junction
+		(at 107.95 71.12)
+		(diameter 0)
+		(color 0 0 0 0)
+	)
+	(junction
 		(at 39.37 45.72)
 		(diameter 0)
@@
 	)
 	(junction
-		(at 115.57 100.33)
+		(at 212.09 123.19)
 		(diameter 0)
 		(color 0 0 0 0)
 	)
 	(junction
-		(at 212.09 123.19)
+		(at 107.95 78.74)
 		(diameter 0)
 		(color 0 0 0 0)
@@
 	(wire
 		(pts
-			(xy 115.57 95.25) (xy 119.38 95.25)
-		)
-		(stroke
-			(width 0)
-			(type default)
-		)
-	)
-	(wire
-		(pts
 			(xy 39.37 45.72) (xy 43.18 45.72)
 		)
@@
 	(wire
 		(pts
-			(xy 127 95.25) (xy 130.81 95.25)
-		)
-		(stroke
-			(width 0)
-			(type default)
-		)
-	)
-	(wire
-		(pts
 			(xy 104.14 142.24) (xy 87.63 142.24)
 		)
@@
 	(wire
 		(pts
-			(xy 115.57 100.33) (xy 115.57 95.25)
-		)
-		(stroke
-			(width 0)
-			(type default)
-		)
-	)
-	(wire
-		(pts
 			(xy 111.76 100.33) (xy 115.57 100.33)
 		)
@@
 	(wire
 		(pts
+			(xy 107.95 71.12) (xy 114.3 71.12)
+		)
+		(stroke
+			(width 0)
+			(type default)
+		)
+	)
+	(wire
+		(pts
 			(xy 114.3 142.24) (xy 104.14 142.24)
 		)
@@
 	(wire
 		(pts
-			(xy 130.81 95.25) (xy 130.81 99.06)
-		)
-		(stroke
-			(width 0)
-			(type default)
-		)
-	)
-	(wire
-		(pts
 			(xy 110.49 22.86) (xy 39.37 22.86)
 		)
@@
 		(pts
 			(xy 218.44 123.19) (xy 212.09 123.19)
+		)
+		(stroke
+			(width 0)
+			(type default)
+		)
+	)
+	(wire
+		(pts
+			(xy 107.95 78.74) (xy 114.3 78.74)
 		)
 		(stroke
@@
 	(symbol
 		(lib_id "Device:C")
-		(at 123.19 95.25 90)
+		(at 114.3 74.93 180)
 		(unit 1)
 		(exclude_from_sim no)
@@
 		(dnp no)
 		(property "Reference" "C8"
-			(at 122.936 101.092 90)
+			(at 120.142 75.184 90)
 			(effects
 				(font
@@
 		)
 		(property "Value" "10uF"
-			(at 123.19 98.806 90)
+			(at 117.856 74.93 90)
 			(effects
 				(font
@@
 		)
 		(property "Footprint" "Capacitor_SMD:C_0402_1005Metric_Pad0.74x0.62mm_HandSolder"
-			(at 127 94.2848 0)
+			(at 113.3348 71.12 0)
 			(effects
 				(font
@@
 		)
 		(property "Datasheet" "~"
-			(at 123.19 95.25 0)
+			(at 114.3 74.93 0)
 			(effects
 				(font
@@
 		)
 		(property "Description" "Unpolarized capacitor"
-			(at 123.19 95.25 0)
+			(at 114.3 74.93 0)
 			(effects
 				(font
@@
 	(symbol
 		(lib_id "power:GND")
+		(at 130.81 99.06 180)
+		(unit 1)
+		(exclude_from_sim no)
+		(in_bom yes)
+		(on_board yes)
+		(dnp no)
+		(fields_autoplaced yes)
+		(property "Reference" "#PWR028"
+			(at 130.81 92.71 0)
+			(effects
+				(font
+					(size 1.27 1.27)
+				)
+				(hide yes)
+			)
+		)
+		(property "Value" "GND"
+			(at 130.81 93.98 0)
+			(effects
+				(font
+					(size 1.27 1.27)
+				)
+			)
+		)
+		(property "Footprint" ""
+			(at 130.81 99.06 0)
+			(effects
+				(font
+					(size 1.27 1.27)
+				)
+				(hide yes)
+			)
+		)
+		(property "Datasheet" ""
+			(at 130.81 99.06 0)
+			(effects
+				(font
+					(size 1.27 1.27)
+				)
+				(hide yes)
+			)
+		)
+		(property "Description" "Power symbol creates a global label with name \"GND\" , ground"
+			(at 130.81 99.06 0)
+			(effects
+				(font
+					(size 1.27 1.27)
+				)
+				(hide yes)
+			)
+		)
+		(pin "1"
+		)
+		(instances
+			(project "smallboard"
+				(path "/52b361e8-aef4-4d01-a2a8-4f07eafc0c1a"
+					(reference "#PWR028")
+					(unit 1)
+				)
+			)
+		)
+	)
+	(symbol
+		(lib_id "power:GND")
 		(at 55.88 135.89 270)
 		(unit 1)
@@
 					(unit 1)
 				)
-			)
-		)
-	)
-	(symbol
-		(lib_id "power:GND")
-		(at 130.81 99.06 90)
-		(unit 1)
-		(exclude_from_sim no)
-		(in_bom yes)
-		(on_board yes)
-		(dnp no)
-		(property "Reference" "#PWR028"
-			(at 137.16 99.06 0)
-			(effects
-				(font
-					(size 1.27 1.27)
-				)
-				(hide yes)
-			)
-		)
-		(property "Value" "GND"
-			(at 130.81 97.028 0)
-			(effects
-				(font
-					(size 1.27 1.27)
-				)
-			)
-		)
-		(property "Footprint" ""
-			(at 130.81 99.06 0)
-			(effects
-				(font
-					(size 1.27 1.27)
-				)
-				(hide yes)
-			)
-		)
-		(property "Datasheet" ""
-			(at 130.81 99.06 0)
-			(effects
-				(font
-					(size 1.27 1.27)
-				)
-				(hide yes)
-			)
-		)
-		(property "Description" "Power symbol creates a global label with name \"GND\" , ground"
-			(at 130.81 99.06 0)
-			(effects
-				(font
-					(size 1.27 1.27)
-				)
-				(hide yes)
-			)
-		)
-		(pin "1"
-		)
-		(instances
-			(project "smallboard"
-				(path "/52b361e8-aef4-4d01-a2a8-4f07eafc0c1a"
-					(reference "#PWR028")
-					(unit 1)
-				)
