File: DemoBoard_STM/DemoBoard_STM.kicad_pcb (KiCad board)
At the start: 4 copper layers, 45 x 45 mm, 57 parts, among them J1 USB4110GFA, J6 M55-7101242R, J7 MSD-1-A, J8 Conn_01x17_Pin, SW1 SW_Push, SW2 SW_Push, U1 RP2040, U2 W25Q128JVSIM, U3 MCP2518FDT-E_QBB, U4 TCAN332DCNR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

Commit message: Routed capacitors
Parts:
- removed C1, C2: 15pF, Capacitor_SMD:C_0402_1005Metric_Pad0.74x0.62mm_HandSolder
- removed C10, C11, C13, C4, C5, C6, C7, C8: 100nF, Capacitor_SMD:C_0402_1005Metric_Pad0.74x0.62mm_HandSolder
- removed C14, C15: 18pF, Capacitor_SMD:C_0402_1005Metric_Pad0.74x0.62mm_HandSolder
- removed C3, C9: 1uF, Capacitor_SMD:C_0402_1005Metric_Pad0.74x0.62mm_HandSolder
- removed R2, R4: 27.4, Resistor_SMD:R_0402_1005Metric_Pad0.72x0.64mm_HandSolder
- removed R3, R7: 10k, Resistor_SMD:R_0402_1005Metric_Pad0.72x0.64mm_HandSolder
- removed R5: 1k, Resistor_SMD:R_0402_1005Metric_Pad0.72x0.64mm_HandSolder
- removed SW2: SW_Push, inspireFly:SW_TL1015AF160QG
- removed TP1: 1.2V, TestPoint:TestPoint_Pad_D1.0mm
- removed TP3: 3.3V, TestPoint:TestPoint_Pad_D1.0mm
- removed U2: W25Q128JVSIM, inspireFly:SOIC_128JVSIM_WIN
- removed U3: MCP2518FDT-E_QBB, inspireFly:SON65P450X300X90-15N
- removed Y2: ABM8-20.000MHZ-10-B1U-T, inspireFly:XTAL_ABM8-272-T3
- added C26: 1uF, Capacitor_SMD:C_0402_1005Metric_Pad0.74x0.62mm_HandSolder, F.Cu at (136.9, 58.7)
- added C27: 100nF, Capacitor_SMD:C_0402_1005Metric_Pad0.74x0.62mm_HandSolder, F.Cu at (133.0, 49.6)
- added C28: 100nF, Capacitor_SMD:C_0402_1005Metric_Pad0.74x0.62mm_HandSolder, F.Cu at (133.0, 50.9)
- added C29: 100nF, Capacitor_SMD:C_0402_1005Metric_Pad0.74x0.62mm_HandSolder, F.Cu at (138.3, 46.2)
- added C30: 10uF, Capacitor_SMD:C_0402_1005Metric_Pad0.74x0.62mm_HandSolder, F.Cu at (141.1, 46.2)
- added C31: 100nF, Capacitor_SMD:C_0402_1005Metric_Pad0.74x0.62mm_HandSolder, F.Cu at (146.5, 52.6)
- added C32: 10uF, Capacitor_SMD:C_0402_1005Metric_Pad0.74x0.62mm_HandSolder, F.Cu at (138.3, 45.0)
- added C33: 2.2uF, Capacitor_SMD:C_0402_1005Metric_Pad0.74x0.62mm_HandSolder, F.Cu at (146.2, 48.0)
- added C34: 2.2uF, Capacitor_SMD:C_0402_1005Metric_Pad0.74x0.62mm_HandSolder, F.Cu at (133.1, 53.4)
- added C35: 6.8pF, Capacitor_SMD:C_0402_1005Metric_Pad0.74x0.62mm_HandSolder, F.Cu at (141.5, 59.6)
- added C36: 6.8pF, Capacitor_SMD:C_0402_1005Metric_Pad0.74x0.62mm_HandSolder, F.Cu at (133.8, 58.7)
- added C37: 12pF, Capacitor_SMD:C_0402_1005Metric_Pad0.74x0.62mm_HandSolder, F.Cu at (141.5, 58.4)
- added C38: 12pF, Capacitor_SMD:C_0402_1005Metric_Pad0.74x0.62mm_HandSolder, F.Cu at (136.9, 59.9)
- added C39: 100nF, Capacitor_SMD:C_0402_1005Metric_Pad0.74x0.62mm_HandSolder, F.Cu at (144.1, 58.4)
- added C40: 1uF, Capacitor_SMD:C_0402_1005Metric_Pad0.74x0.62mm_HandSolder, F.Cu at (144.1, 59.6)
- added C41: 100nF, Capacitor_SMD:C_0402_1005Metric_Pad0.74x0.62mm_HandSolder, F.Cu at (127.0, 56.5)
- added D3: PESD3V3U1UL, Diode_SMD:D_SOD-882, F.Cu at (122.3, 44.5)
- added D4: ESDA14V2SC5, Package_TO_SOT_SMD:SOT-23-5, F.Cu at (129.4, 64.5)
- added D5: ESDA14V2SC5, Package_TO_SOT_SMD:SOT-23-5, F.Cu at (125.6, 49.5)
- added L1: 2.2uH, Inductor_SMD:L_0402_1005Metric_Pad0.77x0.64mm_HandSolder, F.Cu at (125.0, 52.1)
- added Y3: 16MHz, Crystal:Crystal_SMD_3225-4Pin_3.2x2.5mm_HandSoldering, F.Cu at (135.2, 63.1)
- U1: value RP2040 -> STM32U375CGT6Q; footprint Package_DFN_QFN:QFN-56-1EP_7x7mm_P0.4mm_EP3.2x3.2mm -> inspireFly:LQFP48_STM
- Y1: value ABM8-272-T3 -> 32.768kHz; footprint inspireFly:XTAL_ABM8-272-T3 -> Crystal:Crystal_SMD_2012-2Pin_2.0x1.2mm_HandSoldering
- moved SW1 9.81 mm to (129.4, 59.2), turned to 0 degrees
- moved Y1 7.02 mm to (140.0, 66.0)
- moved U1 5.75 mm to (139.8, 52.1), turned to 90 degrees
- moved C25 0.81 mm to (145.3, 45.2)
Connections:
- net GPIO_10 renamed PA3
- net GPIO_11 renamed PA4
- net GPIO_12 renamed PA5
- net GPIO_13 renamed PA6
- net GPIO_18 renamed PA8
- net GPIO_21 renamed PA11
- net GPIO_8 renamed PA1
- SW1 pad 1: RESET -> GND
- SW1 pad 2: GND -> Net-(D3-K)
- U1 pad 1: +3.3V -> VBAT
- U1 pad 10: +3.3V -> PA0
- U1 pad 12: GPIO_9 -> PA2
- U1 pad 17: GPIO_14 -> PA7
- U1 pad 18: GPIO_15 -> PB0
- U1 pad 19: GND -> PB1
- U1 pad 2: SPI0_MISO -> PC13
- U1 pad 20: Net-(U1-XIN) -> Net-(U1-VLXSMPS)
- U1 pad 21: Net-(U1-XOUT) -> VDD
- U1 pad 22: +3.3V -> GND
- U1 pad 23: +1.2V -> Net-(C33-Pad2)
- U1 pad 24: SWCLK -> GND
- U1 pad 25: SWD -> VDD
- U1 pad 26: RESET -> PB13
- U1 pad 27: GPIO_16 -> PB14
- U1 pad 28: GPIO_17 -> PB15
- U1 pad 3: SPI0_CS_CAN -> Net-(U1-PC14-OSC32_IN)
- U1 pad 30: GPIO_19 -> Net-(J2-VCP_TX)
- U1 pad 31: GPIO_20 -> Net-(J2-VCP_RX)
- U1 pad 33: +3.3V -> PA12
- U1 pad 34: GPIO_22 -> Net-(J2-JTMS/SWDIO)
- U1 pad 35: GPIO_23 -> GND
- U1 pad 36: GPIO_24 -> VDD
- U1 pad 37: GPIO_25 -> Net-(J2-JCLK/SWCLK)
- U1 pad 38: ADC_0 -> Net-(J2-JTDI/NC)
- U1 pad 39: ADC_1 -> Net-(J2-JTDO/SWO)
- U1 pad 4: SPI0_CLK -> Net-(U1-PC15-OSC32_OUT)
- U1 pad 40: ADC_2 -> PB4
- U1 pad 41: ADC_3 -> PB5
- U1 pad 42: +3.3V -> PB6
- U1 pad 43: +3.3V -> PB7
- U1 pad 44: +3.3V -> PH3-BOOT0
- U1 pad 45: +1.2V -> PB8
- U1 pad 46: Net-(U1-USB_DM) -> Net-(C33-Pad2)
- U1 pad 47: Net-(U1-USB_DP) -> GND
- U1 pad 48: +3.3V -> VDD
- U1 pad 5: SPI0_MOSI -> Net-(U1-PH0-OSC_IN)
- U1 pad 6: INT_CAN_CONTROLLER -> Net-(U1-PH1-OSC_OUT)
- U1 pad 7: SPI0_CS_SDCARD -> Net-(D3-K)
- U1 pad 8: GPIO_6 -> GND
- U1 pad 9: GPIO_7 -> VDDA
- Y1 pad 1: Net-(U1-XIN) -> Net-(U1-PC15-OSC32_OUT)
- Y1 pad 2: GND -> Net-(U1-PC14-OSC32_IN)
Routing:
- net USB_VOLTAGE: track 53.2 -> 3.51 mm, vias 1 -> 0
- net CAN_HIGH: track 61.4 -> 11.8 mm, vias 1 -> 0
- net CAN_LOW: track 59.8 -> 10.6 mm, vias 3 -> 2
- net GPIO_15: track 42.9 -> 0.00 mm, vias 2 -> 0
- net GPIO_14: track 41.9 -> 0.00 mm, vias 2 -> 1
- net +3.3V: track 49.6 -> 13.6 mm, vias 20 -> 9
- net GND: track 3.85 -> 39.8 mm, vias 16 -> 8
- net GPIO_9: track 35.6 -> 0.00 mm
- net ADC_3: track 35.5 -> 0.00 mm, vias 1 -> 0
- net ADC_2: track 34.0 -> 0.00 mm, vias 1 -> 0
- net ADC_0: track 33.8 -> 0.00 mm, vias 1 -> 0
- net ADC_1: track 33.5 -> 0.00 mm, vias 1 -> 0
- net GPIO_17: track 26.8 -> 0.00 mm, vias 2 -> 0
- net +1.2V: track 24.5 -> 0.00 mm
- net RESET: track 24.1 -> 0.00 mm, vias 2 -> 0
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Other:
- board text removed: "BOOT0"
- board text removed: "RST"
